File: IO_16_8_1/IO_16_8_1.kicad_pcb (KiCad board)
At the start: 2 copper layers, 100 x 100 mm, 224 parts, among them J1 Conn_01x06, J10 Conn_01x06, J11 Conn_01x06, J2 nmount JST 1mm QWIIC, J3 nmount SW Debug, J4 USB_C_Receptacle_USB2.0, J5 Conn_01x06, J6 Conn_01x06, J7 Conn_01x06, J8 Conn_01x06, J9 Conn_01x06, Q1 2N7002, Q10 2N7002, Q11 2N7002, Q12 2N7002, Q13 AO3400A, Q14 AO3400A, Q15 AO3400A, Q16 AO3400A, Q17 2N7002, Q18 2N7002, Q19 2N7002, Q2 2N7002, Q20 2N7002, Q21 2N7002, Q22 2N7002, Q23 2N7002, Q24 2N7002, Q25 IRLR3410, Q26 IRLR3410, Q27 IRLR3410, Q28 IRLR3410, Q29 IRLR3410, Q3 2N7002, Q30 IRLR3410, Q31 IRLR3410, Q32 IRLR3410, Q4 2N7002, Q5 2N7002, Q6 2N7002, Q7 2N7002, Q8 2N7002, Q9 2N7002, SW1 Reset, SW2 Boot, SW3 ADDRESS, U1 ADM3483, U2 W25Q32JVSS, U3 RP2040, U4 LMV321, U5 SN74AHCT1G125, U6 AP2112K-3.3, Y1 12MHz,18pF

Commit message: v010
Parts:
- U2: value W25Q32JVSS -> W25Q128JVSIQ
Changed lines of the file:
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@@
     (pad_to_mask_clearance 0)
     (aux_axis_origin 75 139)
+    (grid_origin 75 139)
     (pcbplotparams
       (layerselection 0x00010fc_ffffffff)
@@
       (viasonmask false)
       (mode 1)
-      (useauxorigin false)
+      (useauxorigin true)
       (hpglpennumber 1)
       (hpglpenspeed 20)
@@
       (effects (font (size 1 1) (thickness 0.15)))
     )
-    (fp_text value "W25Q32JVSS" (at 0 3.56) (layer "F.Fab")
+    (fp_text value "W25Q128JVSIQ" (at 0 3.56) (layer "F.Fab")
       (effects (font (size 1 1) (thickness 0.15)))
     )
@@
     (effects (font (size 5 5) (thickness 1)))
   )
-  (target plus (at 75 139) (size 5) (width 0.1) (layer "Edge.Cuts"))
   (segment (start 140.97 60.96) (end 142.766 59.164) (width 0.2) (layer "F.Cu") (net 1))
   (segment (start 95.3855 117.124) (end 95.855 117.124) (width 0.2) (layer "F.Cu") (net 1))

Commit message: changed R17
Parts:
- R17: value 2k -> 5k
Changed lines of the file:
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@@
       (effects (font (size 1 1) (thickness 0.15)))
     )
-    (fp_text value "2k" (at 0 1.43 90) (layer "F.Fab")
+    (fp_text value "5k" (at 0 1.43 90) (layer "F.Fab")
       (effects (font (size 1 1) (thickness 0.15)))
     )
