File: IO_16_8_1/IO_16_8_1.kicad_pcb (KiCad board)
At the start: 2 copper layers, 100 x 100 mm, 224 parts, among them J1 Conn_01x06, J10 Conn_01x06, J11 Conn_01x06, J2 nmount JST 1mm QWIIC, J3 nmount SW Debug, J4 USB_C_Receptacle_USB2.0, J5 Conn_01x06, J6 Conn_01x06, J7 Conn_01x06, J8 Conn_01x06, J9 Conn_01x06, Q1 2N7002, Q10 2N7002, Q11 2N7002, Q12 2N7002, Q13 AO3400A, Q14 AO3400A, Q15 AO3400A, Q16 AO3400A, Q17 2N7002, Q18 2N7002, Q19 2N7002, Q2 2N7002, Q20 2N7002, Q21 2N7002, Q22 2N7002, Q23 2N7002, Q24 2N7002, Q25 IRLR3410, Q26 IRLR3410, Q27 IRLR3410, Q28 IRLR3410, Q29 IRLR3410, Q3 2N7002, Q30 IRLR3410, Q31 IRLR3410, Q32 IRLR3410, Q4 2N7002, Q5 2N7002, Q6 2N7002, Q7 2N7002, Q8 2N7002, Q9 2N7002, SW1 Reset, SW2 Boot, SW3 ADDRESS, U1 ADM3483, U2 W25Q128JVSIQ, U3 RP2040, U4 LMV321, U5 SN74AHCT1G125, U6 AP2112K-3.3, Y1 12MHz,18pF

Commit message: v101
Parts:
- C29, C30: value nmount -> 470p
Changed lines of the file:
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@@
       (effects (font (size 1 1) (thickness 0.15)))
     )
-    (fp_text value "nmount" (at 3.897 0.091) (layer "F.Fab")
+    (fp_text value "470p" (at 3.897 0.091) (layer "F.Fab")
       (effects (font (size 1 1) (thickness 0.15)))
     )
@@
       (effects (font (size 1 1) (thickness 0.15)))
     )
-    (fp_text value "nmount" (at 4.024 0.091) (layer "F.Fab")
+    (fp_text value "470p" (at 4.024 0.091) (layer "F.Fab")
       (effects (font (size 1 1) (thickness 0.15)))
     )

Commit message: Release 1.1.0
Parts:
- removed F1: T500mA,<0.3Ω, Fuse:Fuse_1206_3216Metric
- added D16: 1A, Diode_SMD:D_SOD-323, F.Cu at (141.0, 53.9)
- added JP1: Jumper_2_Open, Connector_PinHeader_2.54mm:PinHeader_1x02_P2.54mm_Vertical, F.Cu at (113.1, 52.6)
- added JP2: Jumper_2_Open, Connector_PinHeader_2.54mm:PinHeader_1x02_P2.54mm_Vertical, F.Cu at (113.1, 50.1)
- added JP3: Jumper_2_Open, Connector_PinHeader_2.54mm:PinHeader_1x02_P2.54mm_Vertical, F.Cu at (115.6, 47.6)
- C25: value 1000µ 10V -> 100µ 16V; footprint Capacitor_THT:CP_Radial_D10.0mm_P5.00mm -> Capacitor_SMD:CP_Elec_6.3x5.4
- R3, R5: value 1k -> 620
- moved R5 12.2 mm to (112.8, 44.5), turned to 90 degrees
- moved C25 5.06 mm to (122.0, 52.6)
- moved D1 3.44 mm to (108.8, 54.7), turned to -90 degrees
- moved D2 2.08 mm to (106.7, 54.7), turned to -90 degrees
- moved R2 1.41 mm to (104.7, 54.5)
- moved R97 1.21 mm to (118.6, 48.1)
- moved C1 1.15 mm to (103.4, 54.5)
- moved R4 1.09 mm to (111.8, 55.8), turned to 0 degrees
- moved R3 0.78 mm to (114.0, 55.6), turned to 90 degrees
- moved C8 0.72 mm to (116.1, 45.8)
- moved C22 0.20 mm to (126.2, 49.0)
- moved R96 0.20 mm to (118.6, 46.5)
Connections:
- J1 pad 4: GND -> /A
- J1 pad 5: GND -> /B
- J8 pad 5: +5V -> GND
- R3 pad 2: /A -> Net-(R3-Pad2)
- R4 pad 2: /B -> Net-(R4-Pad2)
- R5 pad 1: /B -> Net-(R5-Pad1)
Routing:
- net /B: track 27.8 -> 51.8 mm, vias 2 -> 3
- net /A: track 27.1 -> 49.4 mm
- net +5V: track 200.4 -> 184.8 mm, vias 22 -> 24
- net Net-(R4-Pad2): track 0.00 -> 7.32 mm
- net GND: track 234.0 -> 229.1 mm, vias 287 -> 299
- net Net-(R5-Pad1): track 0.00 -> 4.07 mm
- net Net-(R3-Pad2): track 0.00 -> 3.54 mm
- net +3V3: track 333.3 -> 332.5 mm, vias 32 -> 31
- net /485_RX: track 55.0 -> 55.7 mm

Commit message: changed MOSFETs
Parts:
- Q25, Q26, Q27, Q28, Q29, Q30, Q31, Q32: value IRLR3410 -> NCE0140KA
Changed lines of the file:
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@@
   (title_block
     (title "IO_16_8_1")
-    (date "2024-10-04")
-    (rev "1.1.0")
+    (date "2024-11-16")
+    (rev "1.1.1")
   )
   (layers
@@
   (net 128 "Net-(D13-Pad2)")
   (net 129 "Net-(D14-Pad2)")
-  (net 130 "Net-(R3-Pad2)")
-  (net 131 "Net-(R4-Pad2)")
-  (net 132 "Net-(R5-Pad1)")
+  (net 130 "Net-(JP1-Pad2)")
+  (net 131 "Net-(JP2-Pad2)")
+  (net 132 "Net-(JP3-Pad1)")
   (footprint "Resistor_SMD:R_0603_1608Metric" (layer "F.Cu")
     (at 93.178 75.148 -90)
@@
       (effects (font (size 1 1) (thickness 0.15)))
     )
-    (fp_text value "IRLR3410" (at 1.386 -1.546) (layer "F.Fab")
+    (fp_text value "NCE0140KA" (at 1.386 -1.546) (layer "F.Fab")
       (effects (font (size 1 1) (thickness 0.15)))
     )
@@
       (effects (font (size 1 1) (thickness 0.15)))
     )
-    (fp_text value "IRLR3410" (at 1.132 -1.765) (layer "F.Fab")
+    (fp_text value "NCE0140KA" (at 1.132 -1.765) (layer "F.Fab")
       (effects (font (size 1 1) (thickness 0.15)))
     )
@@
       (net 28 "/A") (pinfunction "A") (pintype "passive"))
     (pad "2" thru_hole oval (at 0 2.54 90) (size 1.7 1.7) (drill 1) (layers *.Cu *.Mask)
-      (net 130 "Net-(R3-Pad2)") (pinfunction "B") (pintype "passive"))
+      (net 130 "Net-(JP1-Pad2)") (pinfunction "B") (pintype "passive"))
     (model "${KICAD6_3DMODEL_DIR}/Connector_PinHeader_2.54mm.3dshapes/PinHeader_1x02_P2.54mm_Vertical.wrl"
       (offset (xyz 0 0 0))
@@
       (effects (font (size 1 1) (thickness 0.15)))
     )
-    (fp_text value "IRLR3410" (at 1.132 -1.983) (layer "F.Fab")
+    (fp_text value "NCE0140KA" (at 1.132 -1.983) (layer "F.Fab")
       (effects (font (size 1 1) (thickness 0.15)))
     )
@@
       (effects (font (size 1 1) (thickness 0.15)))
     )
-    (fp_text value "IRLR3410" (at 0.751 -1.764) (layer "F.Fab")
+    (fp_text value "NCE0140KA" (at 0.751 -1.764) (layer "F.Fab")
       (effects (font (size 1 1) (thickness 0.15)))
     )
@@
       (net 8 "+5V") (pintype "passive"))
     (pad "2" smd roundrect (at 0.51 0 90) (size 0.54 0.64) (layers "F.Cu" "F.Paste" "F.Mask") (roundrect_rratio 0.25)
-      (net 130 "Net-(R3-Pad2)") (pintype "passive"))
+      (net 130 "Net-(JP1-Pad2)") (pintype "passive"))
     (model "${KICAD6_3DMODEL_DIR}/Resistor_SMD.3dshapes/R_0402_1005Metric.wrl"
       (offset (xyz 0 0 0))
@@
       (effects (font (size 1 1) (thickness 0.15)))
     )
-    (fp_text value "IRLR3410" (at 0.878 -1.857) (layer "F.Fab")
+    (fp_text value "NCE0140KA" (at 0.878 -1.857) (layer "F.Fab")
       (effects (font (size 1 1) (thickness 0.15)))
     )
@@
       (effects (font (size 1 1) (thickness 0.15)))
     )
-    (fp_text value "IRLR3410" (at 0.751 -1.671) (layer "F.Fab")
+    (fp_text value "NCE0140KA" (at 0.751 -1.671) (layer "F.Fab")
       (effects (font (size 1 1) (thickness 0.15)))
     )
@@
       (net 121 "/B") (pinfunction "A") (pintype "passive"))
     (pad "2" thru_hole oval (at 0 2.54 90) (size 1.7 1.7) (drill 1) (layers *.Cu *.Mask)
-      (net 131 "Net-(R4-Pad2)") (pinfunction "B") (pintype "passive"))
+      (net 131 "Net-(JP2-Pad2)") (pinfunction "B") (pintype "passive"))
     (model "${KICAD6_3DMODEL_DIR}/Connector_PinHeader_2.54mm.3dshapes/PinHeader_1x02_P2.54mm_Vertical.wrl"
       (offset (xyz 0 0 0))
@@
     (fp_line (start 1.27 -1.27) (end 1.27 3.81) (layer "F.Fab") (width 0.1))
     (pad "1" thru_hole rect (at 0 0 270) (size 1.7 1.7) (drill 1) (layers *.Cu *.Mask)
-      (net 132 "Net-(R5-Pad1)") (pinfunction "A") (pintype "passive"))
+      (net 132 "Net-(JP3-Pad1)") (pinfunction "A") (pintype "passive"))
     (pad "2" thru_hole oval (at 0 2.54 270) (size 1.7 1.7) (drill 1) (layers *.Cu *.Mask)
       (net 121 "/B") (pinfunction "B") (pintype "passive"))
@@
     (fp_line (start -0.525 -0.27) (end 0.525 -0.27) (layer "F.Fab") (width 0.1))
     (pad "1" smd roundrect (at -0.51 0 90) (size 0.54 0.64) (layers "F.Cu" "F.Paste" "F.Mask") (roundrect_rratio 0.25)
-      (net 132 "Net-(R5-Pad1)") (pintype "passive"))
+      (net 132 "Net-(JP3-Pad1)") (pintype "passive"))
     (pad "2" smd roundrect (at 0.51 0 90) (size 0.54 0.64) (layers "F.Cu" "F.Paste" "F.Mask") (roundrect_rratio 0.25)
       (net 1 "GND") (pintype "passive"))
@@
       (net 28 "/A") (pintype "passive"))
     (pad "2" smd roundrect (at 0.825 0) (size 0.8 0.95) (layers "F.Cu" "F.Paste" "F.Mask") (roundrect_rratio 0.25)
-      (net 131 "Net-(R4-Pad2)") (pintype "passive"))
+      (net 131 "Net-(JP2-Pad2)") (pintype "passive"))
     (model "${KICAD6_3DMODEL_DIR}/Resistor_SMD.3dshapes/R_0603_1608Metric.wrl"
       (offset (xyz 0 0 0))
@@
       (effects (font (size 1 1) (thickness 0.15)))
     )
-    (fp_text value "IRLR3410" (at 0.624 -1.926) (layer "F.Fab")
+    (fp_text value "NCE0140KA" (at 0.624 -1.926) (layer "F.Fab")
       (effects (font (size 1 1) (thickness 0.15)))
     )
@@
       (effects (font (size 1 1) (thickness 0.15)))
     )
-    (fp_text value "IRLR3410" (at 0.878 -1.89) (layer "F.Fab")
+    (fp_text value "NCE0140KA" (at 0.878 -1.89) (layer "F.Fab")
       (effects (font (size 1 1) (thickness 0.15)))
     )

Commit message: added production data
Other:
- rule pad_to_mask_clearance: 0 -> 0.05
Changed lines of the file:
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@@
       (dielectric_constraints no)
     )
-    (pad_to_mask_clearance 0)
+    (pad_to_mask_clearance 0.05)
     (aux_axis_origin 75 139)
     (grid_origin 75 139)
@@
     (property "Sheetfile" "IN16.kicad_sch")
     (property "Sheetname" "IN16")
-    (property "exclude_from_bom" "")
-    (attr smd exclude_from_bom)
+    (attr smd)
     (fp_text reference "C30" (at 0 -1.43) (layer "F.SilkS") hide
       (effects (font (size 1 1) (thickness 0.15)))
@@
     (descr "SMD 4x-dip-switch SPST , Slide, row spacing 8.61 mm (338 mils), body size 6.7x11.72mm (see e.g. https://www.ctscorp.com/wp-content/uploads/219.pdf), SMD, LowProfile")
     (tags "SMD DIP Switch SPST Slide 8.61mm 338mil SMD LowProfile")
+    (property "JLCPCB Rotation Offset" "90")
     (property "Sheetfile" "IO_16_8_1.kicad_sch")
     (property "Sheetname" "")
@@
     (descr "QFN, 56 Pin (https://datasheets.raspberrypi.com/rp2040/rp2040-datasheet.pdf#page=634), generated with kicad-footprint-generator ipc_noLead_generator.py")
     (tags "QFN NoLead")
+    (property "JLCPCB Rotation Offset" "-90")
     (property "Sheetfile" "IO_16_8_1.kicad_sch")
     (property "Sheetname" "")
@@
     (property "Sheetfile" "IN16.kicad_sch")
     (property "Sheetname" "IN16")
-    (property "exclude_from_bom" "")
-    (attr smd exclude_from_bom)
+    (attr smd)
     (fp_text reference "C29" (at 0 -1.43) (layer "F.SilkS") hide
       (effects (font (size 1 1) (thickness 0.15)))
@@
     (descr "SOT, 5 Pin (https://www.jedec.org/sites/default/files/docs/Mo-178c.PDF variant AA), generated with kicad-footprint-generator ipc_gullwing_generator.py")
     (tags "SOT TO_SOT_SMD")
+    (property "JLCPCB Rotation Offset" "90")
     (property "Sheetfile" "IO_16_8_1.kicad_sch")
     (property "Sheetname" "")
@@
     (property "Sheetfile" "IO_16_8_1.kicad_sch")
     (property "Sheetname" "")
-    (attr through_hole)
+    (property "exclude_from_bom" "")
+    (attr through_hole exclude_from_bom)
     (fp_text reference "TP2" (at 0 2.25) (layer "F.SilkS")
       (effects (font (size 1 1) (thickness 0.15)))
@@
     (property "Sheetfile" "IO_16_8_1.kicad_sch")
     (property "Sheetname" "")
-    (attr through_hole)
+    (property "exclude_from_bom" "")
+    (attr through_hole exclude_from_bom)
     (fp_text reference "TP1" (at 0.127 -2.159) (layer "F.SilkS")
       (effects (font (size 1 1) (thickness 0.15)))
@@
     (descr "SMD capacitor, aluminum electrolytic, Panasonic C55, 6.3x5.4mm")
     (tags "capacitor electrolytic")
+    (property "JLCPCB Rotation Offset" "180")
     (property "Sheetfile" "IO_16_8_1.kicad_sch")
     (property "Sheetname" "")
