File: IO_16_8_1/IN16.kicad_sch (KiCad schematic)
At the start: 98 parts, among them J6 Conn_01x06, J7 Conn_01x06, J8 Conn_01x06, Q1 2N7002, Q10 2N7002, Q11 2N7002, Q12 2N7002, Q13 AO3400A, Q14 AO3400A, Q15 AO3400A, Q16 AO3400A, Q17 2N7002, Q18 2N7002, Q19 2N7002, Q2 2N7002, Q20 2N7002, Q21 2N7002, Q22 2N7002, Q23 2N7002, Q24 2N7002, Q3 2N7002, Q4 2N7002, Q5 2N7002, Q6 2N7002, Q7 2N7002, Q8 2N7002, Q9 2N7002

Commit message: v101
Parts:
- C29, C30: value nmount -> 470p
Other:
- note added: "Remove C29+C30 when using fast serial transmission. Resolder R34 to R99 and R35 to R98 when using 3.3V serial voltage level."
Changed lines of the file:
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@@
     (effects (font (size 3 3) (thickness 0.6) bold) (justify left bottom))
+  )
+  (text "Remove C29+C30\nwhen using fast\nserial transmission.\n\nResolder\nR34 to R99 and\nR35 to R98 when \nusing 3.3V serial\nvoltage level."
+    (at 62.23 120.65 0)
+    (effects (font (size 1.27 1.27)) (justify left bottom))
   )
   (text "4" (at 123.19 172.72 0)
@@
       (effects (font (size 1.27 1.27)) (justify left))
     )
-    (property "Value" "nmount" (id 1) (at 81.28 102.87 90)
+    (property "Value" "470p" (id 1) (at 81.28 102.87 90)
       (effects (font (size 1.27 1.27)) (justify left))
     )
@@
       (effects (font (size 1.27 1.27)) (justify left))
     )
-    (property "Value" "nmount" (id 1) (at 81.28 138.43 90)
-      (effects (font (size 1.27 1.27)) (justify left))
-    )
+    (property "Value" "470p" (id 1) (at 81.28 138.43 90)
+      (effects (font (size 1.27 1.27)) (justify left))
+    )

Commit message: Release 1.1.0
Connections:
- net +5V: no longer J8.5 (Pin_5)
- net GND: now also J8.5 (Pin_5)
Other:
- title: Inputs, Low Power Outputs -> IO_16_8_1
Changed lines of the file:
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@@
   (paper "A3")
   (title_block
-    (title "Inputs, Low Power Outputs")
-    (date "2023-01-29")
-    (rev "1.0.0")
+    (title "IO_16_8_1")
+    (date "2024-10-04")
+    (rev "1.1.0")
   )
   (junction (at 105.41 170.18) (diameter 0) (color 0 0 0 0)
@@
   (junction (at 365.76 146.05) (diameter 0) (color 0 0 0 0)
   )
+  (junction (at 274.32 160.02) (diameter 0) (color 0 0 0 0)
+  )
   (junction (at 105.41 48.26) (diameter 0) (color 0 0 0 0)
   )
@@
   (junction (at 189.23 170.18) (diameter 0) (color 0 0 0 0)
   )
-  (junction (at 283.21 162.56) (diameter 0) (color 0 0 0 0)
-  )
   (junction (at 209.55 209.55) (diameter 0) (color 0 0 0 0)
   )
@@
     (stroke (width 0) (type default) (color 0 0 0 0))
   )
-  (wire (pts (xy 283.21 161.29) (xy 283.21 162.56))
+  (wire (pts (xy 283.21 161.29) (xy 283.21 163.83))
     (stroke (width 0) (type default) (color 0 0 0 0))
   )
@@
     (stroke (width 0) (type default) (color 0 0 0 0))
   )
-  (wire (pts (xy 276.86 162.56) (xy 283.21 162.56))
-    (stroke (width 0) (type default) (color 0 0 0 0))
-  )
   (wire (pts (xy 97.79 48.26) (xy 105.41 48.26))
     (stroke (width 0) (type default) (color 0 0 0 0))
@@
     (stroke (width 0) (type default) (color 0 0 0 0))
   )
+  (wire (pts (xy 274.32 157.48) (xy 274.32 160.02))
+    (stroke (width 0) (type default) (color 0 0 0 0))
+  )
   (wire (pts (xy 365.76 168.91) (xy 367.03 168.91))
     (stroke (width 0) (type default) (color 0 0 0 0))
@@
     (stroke (width 0) (type default) (color 0 0 0 0))
   )
-  (wire (pts (xy 270.51 157.48) (xy 276.86 157.48))
-    (stroke (width 0) (type default) (color 0 0 0 0))
-  )
   (wire (pts (xy 85.09 96.52) (xy 85.09 95.25))
     (stroke (width 0) (type default) (color 0 0 0 0))
@@
     (stroke (width 0) (type default) (color 0 0 0 0))
   )
-  (wire (pts (xy 283.21 162.56) (xy 283.21 163.83))
-    (stroke (width 0) (type default) (color 0 0 0 0))
-  )
   (wire (pts (xy 105.41 58.42) (xy 102.87 58.42))
     (stroke (width 0) (type default) (color 0 0 0 0))
@@
     (stroke (width 0) (type default) (color 0 0 0 0))
   )
-  (wire (pts (xy 276.86 157.48) (xy 276.86 162.56))
-    (stroke (width 0) (type default) (color 0 0 0 0))
-  )
   (wire (pts (xy 358.14 85.09) (xy 365.76 85.09))
     (stroke (width 0) (type default) (color 0 0 0 0))
@@
     (stroke (width 0) (type default) (color 0 0 0 0))
   )
+  (wire (pts (xy 270.51 157.48) (xy 274.32 157.48))
+    (stroke (width 0) (type default) (color 0 0 0 0))
+  )

Commit message: added production data
Parts:
- C29, C30: now in the parts list
Changed lines of the file:
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@@
   )
   (symbol (lib_id "Device:C") (at 85.09 100.33 0) (mirror y) (unit 1)
-    (in_bom no) (on_board yes)
+    (in_bom yes) (on_board yes)
     (property "Reference" "C29" (id 0) (at 86.36 99.06 90)
       (effects (font (size 1.27 1.27)) (justify left))
@@
   )
   (symbol (lib_id "Device:C") (at 85.09 135.89 0) (mirror y) (unit 1)
-    (in_bom no) (on_board yes)
+    (in_bom yes) (on_board yes)
     (property "Reference" "C30" (id 0) (at 86.36 134.62 90)
       (effects (font (size 1.27 1.27)) (justify left))
