File: IO_16_8_1/IO_16_8_1.kicad_sch (KiCad schematic)
At the start: 78 parts, among them J1 Conn_01x06, J2 nmount JST 1mm QWIIC, J3 nmount SW Debug, J4 USB_C_Receptacle_USB2.0, J5 Conn_01x06, SW1 Reset, SW2 Boot, SW3 ADDRESS, U1 ADM3483, U2 W25Q128JVSIQ, U3 RP2040, U4 LMV321, U5 SN74AHCT1G125, U6 AP2112K-3.3, Y1 12MHz,18pF

Commit message: Release 1.1.0
Parts:
- removed F1: T500mA,<0.3Ω, Fuse:Fuse_1206_3216Metric, symbol Device:Fuse
- added D16: 1A, Diode_SMD:D_SOD-323, symbol Device:D_Schottky
- added JP1, JP2, JP3: Jumper_2_Open, Connector_PinHeader_2.54mm:PinHeader_1x02_P2.54mm_Vertical, symbol Jumper:Jumper_2_Open
- C25: value 1000µ 10V -> 100µ 16V; footprint Capacitor_THT:CP_Radial_D10.0mm_P5.00mm -> Capacitor_SMD:CP_Elec_6.3x5.4
- R3, R5: value 1k -> 620
Connections:
- net +5V: now also D16.1 (K)
- net 5V_IN: now also D16.2 (A)
- net A: now also J1.4 (Pin_4), JP1.1 (A); no longer R3.2
- net B: now also J1.5 (Pin_5), JP2.1 (A), JP3.2 (B); no longer R4.2, R5.1
- net GND: no longer J1.4 (Pin_4), J1.5 (Pin_5)
- new net: JP3.1 (A), R5.1
- new net: JP1.2 (B), R3.2
- new net: JP2.2 (B), R4.2
Other:
- moved on the sheet: C1, D1, D2, R2, R3, R4, R5

Commit message: added production data
Parts:
- C25: JLCPCB Rotation Offset (none) -> 180
- SW3, U6: JLCPCB Rotation Offset (none) -> 90
- TP1, TP2: now left out of the parts list
- U3: JLCPCB Rotation Offset (none) -> -90
Changed lines of the file:
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@@
+      (effects (font (size 1.27 1.27)) hide)
+    )
+    (property "JLCPCB Rotation Offset" "90" (id 4) (at 321.31 31.75 0)
       (effects (font (size 1.27 1.27)) hide)
     )
@@
       (effects (font (size 1.27 1.27)) hide)
     )
+    (property "JLCPCB Rotation Offset" "90" (id 4) (at 250.19 214.63 0)
+      (effects (font (size 1.27 1.27)) hide)
+    )
     (pin "1")
     (pin "2")
@@
       (effects (font (size 1.27 1.27)) hide)
     )
+    (property "JLCPCB Rotation Offset" "180" (id 4) (at 334.01 99.06 0)
+      (effects (font (size 1.27 1.27)) hide)
+    )
     (pin "1")
     (pin "2")
@@
   )
   (symbol (lib_id "Connector:TestPoint") (at 261.62 160.02 0) (unit 1)
-    (in_bom yes) (on_board yes) (fields_autoplaced)
+    (in_bom no) (on_board yes) (fields_autoplaced)
     (property "Reference" "TP1" (id 0) (at 264.16 155.4479 0)
       (effects (font (size 1.27 1.27)) (justify left))
@@
   )
   (symbol (lib_id "Connector:TestPoint") (at 284.48 160.02 0) (unit 1)
-    (in_bom yes) (on_board yes) (fields_autoplaced)
+    (in_bom no) (on_board yes) (fields_autoplaced)
     (property "Reference" "TP2" (id 0) (at 287.02 155.4479 0)
       (effects (font (size 1.27 1.27)) (justify left))
@@
       (effects (font (size 1.27 1.27)) hide)
     )
+    (property "JLCPCB Rotation Offset" "-90" (id 4) (at 195.58 134.62 0)
+      (effects (font (size 1.27 1.27)) hide)
+    )
